File: Daughter Board/Volterra Doughter Board MKS GEN L 2.1.sch (EAGLE design)
At the start: 52 parts, among them J14 FEMALE 2x3, J5 455-1750-1-ND, J6 455-1750-1-ND, J7 455-1750-1-ND, K1 FFC/FPC/34PIN/1MMPITCH/TOPLOCK, X10 FIL_HEAT, X11 FIL_THM, X12 CH_THM, X13 CH_HEAT, X14 24V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

Commit message: MKS GEN L 2.1
CHANGES MADE
Parts:
- added U$2: MAKEININDIA, FracktalWorks_Eagle_Library:MAKEININDIA
- X8: value JST-XH-04-PIN-LONG-PAD -> AUTO BED LEVELING
Changed lines of the file:
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@@
 <part name="X9" library="Rembrandt Electronics - JST XH Connectors v1-0" deviceset="JST-XH-02-PIN" device="-LONG-PAD" value="Y_LMT"/>
 <part name="HEADER" library="SparkFun-Connectors" deviceset="CONN_03" device="" value="455-1750-1-ND"/>
-<part name="X8" library="Rembrandt Electronics - JST XH Connectors v1-0" deviceset="JST-XH-04-PIN" device="-LONG-PAD">
+<part name="X8" library="Rembrandt Electronics - JST XH Connectors v1-0" deviceset="JST-XH-04-PIN" device="-LONG-PAD" value="AUTO BED LEVELING">
 <attribute name="AUTOBEDLEVL" value="AUTO BED LEVEL"/>
 </part>
 <part name="X14" library="Rembrandt Electronics - JST XH Connectors v1-0" deviceset="JST-XH-02-PIN" device="-LONG-PAD" value="24V"/>
+<part name="U$2" library="FracktalWorks_Eagle_Library" deviceset="MAKEININDIA" device=""/>
 </parts>
 <sheets>
@@
 <attribute name="VALUE" x="364.363" y="255.778" size="1.778" layer="96" rot="R90"/>
 </instance>
+<instance part="U$2" gate="G$1" x="408.94" y="43.18" smashed="yes"/>
 </instances>
 <busses>
