File: Daughter Board/Volterra Doughter Board MKS GEN L 2.1.brd (EAGLE design)
At the start: 92.8 x 61 mm, 52 parts, among them J14 FEMALE 2x3, J5 455-1750-1-ND, J6 455-1750-1-ND, J7 455-1750-1-ND, K1 FFC/FPC/34PIN/1MMPITCH/TOPLOCK, X10 FIL_HEAT, X11 FIL_THM, X12 CH_THM, X13 CH_HEAT, X14 24V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

Commit message: MKS GEN L 2.1
CHANGES MADE
Parts:
- added U$2: MAKEININDIA, FracktalWorks_Eagle_Library:MAKEININDIA
- X8: value JST-XH-04-PIN-LONG-PAD -> AUTO BED LEVELING
- moved TP19 35.4 mm to (74.5, 9.53)
- moved TP17 30.9 mm to (74.4, 17.1)
- moved TP20 27.0 mm to (71.0, 9.53)
- moved TP18 25.8 mm to (70.5, 17.3)
- moved TP22 23.7 mm to (74.5, 13.6)
- moved TP23 22.3 mm to (70.6, 13.5)
Routing:
- net CF+: track 31.8 -> 69.8 mm
- net H1-: track 82.3 -> 112.9 mm
- net CF-: track 32.3 -> 60.2 mm
- net H0-: track 80.4 -> 104.7 mm
- net H0+: track 65.8 -> 88.0 mm, vias 3 -> 4
- net H1+: track 76.1 -> 86.8 mm, vias 3 -> 4
- net A0+: track 12.8 -> 14.6 mm
- added copper zone on layer 1, net GND
- added copper zone on layer 16, net GND
Other:
- board size 92.8 x 61 mm -> 92.8 x 60.6 mm
- board text added: "24V"
- board text added: "5V"
- board text added: "BLACK"
- board text added: "BROWN"
- board text added: "CH_HEAT"
- board text added: "GND"
- board text added: "PT0"
- board text added: "PT1"
- board text added: "SERVO_DAT"
- board text added: "X_LIM"
- board text added: "Y_LIM"
- board text added: "Z_DIR"
- board text added: "Z_OUT"

Commit message: update
Parts:
- moved FRAME1 14.0 mm to (41.9, -14.0)
Other:
- board text added: "A GAUTHAM"
- board text added: "DESIGNED BY"
Changed lines of the file:
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@@
 <grid distance="50" unitdist="mil" unit="mil" style="lines" multiple="1" display="no" altdistance="5" altunitdist="mil" altunit="mil"/>
 <layers>
-<layer number="1" name="Top" color="4" fill="1" visible="no" active="yes"/>
+<layer number="1" name="Top" color="4" fill="1" visible="yes" active="yes"/>
 <layer number="2" name="Route2" color="16" fill="1" visible="no" active="no"/>
 <layer number="3" name="Route3" color="17" fill="1" visible="no" active="no"/>
@@
 <layer number="14" name="Route14" color="22" fill="1" visible="no" active="no"/>
 <layer number="15" name="Route15" color="23" fill="1" visible="no" active="no"/>
-<layer number="16" name="Bottom" color="1" fill="1" visible="no" active="yes"/>
+<layer number="16" name="Bottom" color="1" fill="1" visible="yes" active="yes"/>
 <layer number="17" name="Pads" color="2" fill="1" visible="yes" active="yes"/>
 <layer number="18" name="Vias" color="2" fill="1" visible="yes" active="yes"/>
@@
 <layer number="25" name="tNames" color="7" fill="1" visible="yes" active="yes"/>
 <layer number="26" name="bNames" color="7" fill="1" visible="yes" active="yes"/>
-<layer number="27" name="tValues" color="7" fill="1" visible="yes" active="yes"/>
+<layer number="27" name="tValues" color="7" fill="1" visible="no" active="yes"/>
 <layer number="28" name="bValues" color="7" fill="1" visible="no" active="yes"/>
-<layer number="29" name="tStop" color="7" fill="3" visible="yes" active="yes"/>
+<layer number="29" name="tStop" color="7" fill="3" visible="no" active="yes"/>
 <layer number="30" name="bStop" color="7" fill="6" visible="no" active="yes"/>
-<layer number="31" name="tCream" color="7" fill="4" visible="yes" active="yes"/>
+<layer number="31" name="tCream" color="7" fill="4" visible="no" active="yes"/>
 <layer number="32" name="bCream" color="7" fill="5" visible="no" active="yes"/>
-<layer number="33" name="tFinish" color="6" fill="3" visible="yes" active="yes"/>
+<layer number="33" name="tFinish" color="6" fill="3" visible="no" active="yes"/>
 <layer number="34" name="bFinish" color="6" fill="6" visible="no" active="yes"/>
-<layer number="35" name="tGlue" color="7" fill="4" visible="yes" active="yes"/>
+<layer number="35" name="tGlue" color="7" fill="4" visible="no" active="yes"/>
 <layer number="36" name="bGlue" color="7" fill="5" visible="no" active="yes"/>
-<layer number="37" name="tTest" color="7" fill="1" visible="yes" active="yes"/>
+<layer number="37" name="tTest" color="7" fill="1" visible="no" active="yes"/>
 <layer number="38" name="bTest" color="7" fill="1" visible="no" active="yes"/>
 <layer number="39" name="tKeepout" color="4" fill="11" visible="yes" active="yes"/>
@@
 <text x="63.5" y="4.064" size="1.27" layer="25">H1-</text>
 <text x="58.674" y="4.064" size="1.27" layer="25">H1+</text>
-<text x="43.434" y="3.556" size="0.3048" layer="25" font="vector">BROWN</text>
-<text x="38.227" y="3.556" size="0.3048" layer="25" font="vector">BLACK</text>
+<text x="43.434" y="3.556" size="0.508" layer="25" font="vector">BROWN</text>
+<text x="38.227" y="3.556" size="0.508" layer="25" font="vector">BLACK</text>
 <text x="100.076" y="49.276" size="1.016" layer="25">24V</text>
 <text x="106.807" y="49.276" size="1.016" layer="25">Z_DIR</text>
@@
 <text x="106.426" y="36.83" size="1.016" layer="25">Y_LIM</text>
 <text x="97.663" y="32.258" size="1.016" layer="25">SERVO_DAT</text>
+<text x="67.691" y="17.526" size="1.016" layer="25">H1+</text>
+<text x="74.803" y="17.78" size="1.016" layer="25">H1-</text>
+<text x="74.93" y="14.097" size="1.016" layer="25">H0-</text>
+<text x="67.945" y="14.097" size="1.016" layer="25">H0+</text>
+<text x="74.93" y="10.287" size="1.016" layer="25">CF+</text>
+<text x="68.326" y="9.779" size="1.016" layer="25">CF-</text>
+<text x="118.11" y="12.7" size="0.8128" layer="26" rot="MR270">DESIGNED BY</text>
+<text x="116.84" y="11.43" size="0.8128" layer="26" rot="MR270">A GAUTHAM</text>
 </plain>
 <attributes>
@@
 </autorouter>
 <elements>
-<element name="FRAME1" library="SparkFun-Aesthetics" package="CREATIVE_COMMONS" value="FRAME-LEDGER" x="55.88" y="-13.97" smashed="yes"/>
+<element name="FRAME1" library="SparkFun-Aesthetics" package="CREATIVE_COMMONS" value="FRAME-LEDGER" x="41.91" y="-13.97" smashed="yes"/>
 <element name="J1" library="SparkFun-Connectors" package="1X02" value="" x="89.154" y="3.81" smashed="yes">
 <attribute name="NAME" x="87.884" y="5.207" size="0.6096" layer="25" font="vector" ratio="20"/>
@@
 <vertex x="25.654" y="60.071" curve="-90"/>
 </polygon>
+<polygon width="0.0762" layer="1" orphans="yes">
+<vertex x="26.289" y="60.579"/>
+<vertex x="115.824" y="60.579" curve="-90"/>
+<vertex x="118.491" y="57.912"/>
+<vertex x="118.491" y="2.032" curve="-90"/>
+<vertex x="116.459" y="0"/>
+<vertex x="36.957" y="0" curve="-90"/>
+<vertex x="35.56" y="1.397"/>
+<vertex x="35.56" y="15.367" curve="90"/>
+<vertex x="34.417" y="16.51"/>
+<vertex x="27.686" y="16.51" curve="-90"/>
+<vertex x="25.654" y="18.542"/>
+<vertex x="25.654" y="60.071" curve="-90"/>
+<vertex x="26.162" y="60.579"/>
+</polygon>
 </signal>
